Commit message: add collision wart to wrist

File: kuka_lbr_iisy_support/urdf/lbr_iisy15_r930_macro.xacro (robot description, xacro)
@@ -132,4 +132,10 @@
         <origin rpy="-0.0 0.0 -0.0" xyz="0.0 0.0 0.0"/>
       </collision>
+      <collision>
+        <geometry>
+          <box size="0.035 0.035 0.03"/>
+        </geometry>
+        <origin rpy="0.0 0.0 0.0" xyz="0 0.094 -0.144"/>
+      </collision>
       <inertial>
         <inertia ixx="0.00390274036654823" ixy="0.0" ixz="0.0" iyy="0.00286930887521153" iyz="0.0" izz="0.00403512413298348"/>

Commit message: extend collision wart on wrist

File: kuka_lbr_iisy_support/urdf/lbr_iisy15_r930_macro.xacro (robot description, xacro)
@@ -134,5 +134,5 @@
       <collision>
         <geometry>
-          <box size="0.035 0.035 0.03"/>
+          <box size="0.065 0.085 0.065"/>
         </geometry>
         <origin rpy="0.0 0.0 0.0" xyz="0 0.094 -0.144"/>

Commit message: inflate wart & link 3

File: kuka_lbr_iisy_support/urdf/lbr_iisy15_r930_macro.xacro (robot description, xacro)
@@ -68,5 +68,5 @@
       <collision>
         <geometry>
-          <mesh filename="package://${package_name}/meshes/lbr_iisy15_r930/collision/link_3.stl"/>
+          <mesh filename="package://${package_name}/meshes/lbr_iisy15_r930/collision/link_3.stl" scale="1.1 1.1 1.1"/>
         </geometry>
         <origin rpy="-0.0 0.0 -0.0" xyz="0.0 0.0 0.0"/>
@@ -134,5 +134,5 @@
       <collision>
         <geometry>
-          <box size="0.065 0.085 0.065"/>
+          <box size="0.075 0.095 0.065"/>
         </geometry>
         <origin rpy="0.0 0.0 0.0" xyz="0 0.094 -0.144"/>
